File: PCB/FCU_v1/PERIPHERALS.kicad_sch (KiCad schematic)
At the start: 59 parts, among them J2 USB_B_Micro, J4 Conn_Coaxial_Small, U10 SN65HVD232, U3 TLV75533PDYDR, U4 BMI088, U5 LIS2MDL, U6 LPS22HH, U7 W25Q64JV, U8 USBLC6-2SC6, U9 MAX-M10M-20B

Commit message: Update FCU_v1 PCB and add new resistors
Reworked net assignments and added new nets in FCU_v1.kicad_pcb. Added and repositioned resistors R23 and R28, and updated footprints and net connections. Also updated several backup files and made minor schematic changes in MCU.kicad_sch and PERIPHERALS.kicad_sch.
Parts:
- removed J2: USB_B_Micro, Connector_USB:USB_Micro-B_Wuerth_629105150521_CircularHoles, symbol Connector:USB_B_Micro
- added J11: USB_C_Receptacle_USB2.0_16P, Connector_USB:USB_C_Receptacle_GCT_USB4105-xx-A_16P_TopMnt_Horizontal, symbol Connector:USB_C_Receptacle_USB2.0_16P
- added R35, R36: 5k1, Resistor_SMD:R_0603_1608Metric, symbol Device:R
Connections:
- net D+: now also J11.A6 (D+), J11.B6 (D+)
- net D-: now also J11.A7 (D-), J11.B7 (D-)
- net GND: now also C18.2, C19.2, J11.A1 (GND), J11.A12 (GND), J11.B1 (GND), J11.B12 (GND), J11.S1 (SHIELD), R35.1, R36.1
- net USB_VBUS: now reaches D6.1 (A1), FB2.1, U8.5 (VBUS)
- net USB_VBUS: now also J11.A4 (VBUS), J11.A9 (VBUS), J11.B4 (VBUS), J11.B9 (VBUS)
- new net: J11.A5 (CC1), R36.2
- new net: J11.B5 (CC2), R35.2
Other:
- moved on the sheet: C17, C18, C19, C20, D2, D3, D6, FB2, R4, R5, R6, U3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

Commit message: Adjust PCB footprint positions and metadata
Add three FCU_v1 backup archives and apply multiple PCB layout fixes: reposition and reorient many footprints (resistors, capacitors, inductors, diodes, SOT-23, LQFP, LGA, etc.), update pad orientation/rotation entries, and correct numerous fp_line coordinates and UUIDs. Also include small updates to project/prl and PERIPHERALS schematic references. These changes refine component placement and silkscreen/fabrication outlines for the FCU_v1 board.
Parts:
- added C10: 100n, Capacitor_SMD:C_0805_2012Metric, symbol Device:C
Connections:
- net 3V3_FCU: now also C10.1
- net GND: now also C10.2
- no-connect marks 11 -> 12
Other:
- note added: "If I understand correctly we dont have to use active antenna, therefore we use only RF_IN pin without LNA_EN, which I think is for active antennas. But anyway I think we need to match impedance of antenna with RF_IN's which I need to check at what value it is. Maybe we need to add just PI filter for this"
- moved on the sheet: C32
Changed lines of the file:
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@@
 		)
 	)
+	(text "If I understand correctly we dont have to use active antenna,\ntherefore we use only RF_IN pin without LNA_EN, which I think\nis for active antennas.\nBut anyway I think we need to match impedance of antenna\nwith RF_IN's which I need to check at what value it is.\nMaybe we need to add just PI filter for this"
+		(exclude_from_sim no)
+		(at 203.2 35.814 0)
+		(effects
+			(font
+				(size 0.635 0.635)
+				(thickness 0.0794)
+			)
+		)
+	)
 	(text "GNSS\nMAX-M10M-20B"
 		(exclude_from_sim no)
@@
 	)
 	(junction
+		(at 163.83 26.67)
+		(diameter 0)
+		(color 0 0 0 0)
+	)
+	(junction
 		(at 116.84 176.53)
 		(diameter 0)
@@
 	)
 	(junction
-		(at 167.64 26.67)
-		(diameter 0)
-		(color 0 0 0 0)
-	)
-	(junction
 		(at 46.99 90.17)
 		(diameter 0)
@@
 	)
 	(junction
+		(at 163.83 36.83)
+		(diameter 0)
+		(color 0 0 0 0)
+	)
+	(junction
 		(at 114.3 68.58)
 		(diameter 0)
@@
 	)
 	(junction
+		(at 170.18 26.67)
+		(diameter 0)
+		(color 0 0 0 0)
+	)
+	(junction
 		(at 158.75 102.87)
 		(diameter 0)
@@
 	)
 	(no_connect
+		(at 196.85 49.53)
+	)
+	(no_connect
 		(at 116.84 111.76)
 	)
@@
 	(wire
 		(pts
-			(xy 167.64 26.67) (xy 167.64 27.94)
+			(xy 163.83 26.67) (xy 163.83 27.94)
 		)
 		(stroke
@@
 	(wire
 		(pts
-			(xy 167.64 35.56) (xy 167.64 36.83)
+			(xy 163.83 35.56) (xy 163.83 36.83)
 		)
 		(stroke
@@
 	(wire
 		(pts
+			(xy 163.83 26.67) (xy 170.18 26.67)
+		)
+		(stroke
+			(width 0)
+			(type default)
+		)
+	)
+	(wire
+		(pts
 			(xy 128.27 27.94) (xy 134.62 27.94)
 		)
@@
 	(wire
 		(pts
+			(xy 170.18 26.67) (xy 176.53 26.67)
+		)
+		(stroke
+			(width 0)
+			(type default)
+		)
+	)
+	(wire
+		(pts
 			(xy 114.3 185.42) (xy 114.3 187.96)
 		)
@@
 	(wire
 		(pts
+			(xy 163.83 36.83) (xy 170.18 36.83)
+		)
+		(stroke
+			(width 0)
+			(type default)
+		)
+	)
+	(wire
+		(pts
 			(xy 60.96 168.91) (xy 62.23 168.91)
 		)
@@
 	(wire
 		(pts
-			(xy 163.83 26.67) (xy 167.64 26.67)
+			(xy 160.02 26.67) (xy 163.83 26.67)
 		)
 		(stroke
@@
 	(wire
 		(pts
+			(xy 170.18 35.56) (xy 170.18 36.83)
+		)
+		(stroke
+			(width 0)
+			(type default)
+		)
+	)
+	(wire
+		(pts
 			(xy 139.7 151.13) (xy 139.7 152.4)
 		)
@@
 	(wire
 		(pts
-			(xy 167.64 26.67) (xy 176.53 26.67)
+			(xy 46.99 95.25) (xy 46.99 93.98)
 		)
 		(stroke
@@
 	(wire
 		(pts
-			(xy 46.99 95.25) (xy 46.99 93.98)
+			(xy 35.56 90.17) (xy 46.99 90.17)
 		)
 		(stroke
@@
 	(wire
 		(pts
-			(xy 35.56 90.17) (xy 46.99 90.17)
+			(xy 153.67 113.03) (xy 158.75 113.03)
 		)
 		(stroke
@@
 	(wire
 		(pts
-			(xy 153.67 113.03) (xy 158.75 113.03)
+			(xy 69.85 140.97) (xy 69.85 142.24)
 		)
 		(stroke
@@
 	(wire
 		(pts
-			(xy 69.85 140.97) (xy 69.85 142.24)
+			(xy 35.56 90.17) (xy 35.56 91.44)
 		)
 		(stroke
@@
 	(wire
 		(pts
-			(xy 35.56 90.17) (xy 35.56 91.44)
+			(xy 76.2 63.5) (xy 83.82 63.5)
 		)
 		(stroke
@@
 	(wire
 		(pts
-			(xy 76.2 63.5) (xy 83.82 63.5)
+			(xy 170.18 26.67) (xy 170.18 27.94)
 		)
 		(stroke
@@
 	(wire
 		(pts
+			(xy 163.83 38.1) (xy 163.83 36.83)
+		)
+		(stroke
+			(width 0)
+			(type default)
+		)
+	)
+	(wire
+		(pts
 			(xy 100.33 49.53) (xy 101.6 49.53)
 		)
@@
 	(global_label "3V3_FCU"
 		(shape input)
-		(at 163.83 26.67 180)
+		(at 160.02 26.67 180)
 		(fields_autoplaced yes)
 		(effects
@@
 		)
 		(property "Intersheetrefs" "${INTERSHEET_REFS}"
-			(at 152.6805 26.67 0)
+			(at 148.8705 26.67 0)
 			(effects
 				(font
@@
 	(symbol
 		(lib_id "Device:C")
-		(at 167.64 31.75 0)
+		(at 163.83 31.75 0)
 		(unit 1)
 		(exclude_from_sim no)
@@
 		(dnp no)
 		(property "Reference" "C32"
-			(at 163.322 29.21 0)
+			(at 159.512 29.21 0)
 			(effects
 				(font
@@
 		)
 		(property "Value" "100n"
-			(at 162.56 34.036 0)
+			(at 158.75 34.036 0)
 			(effects
 				(font
@@
 		)
 		(property "Footprint" "Capacitor_SMD:C_0805_2012Metric"
-			(at 168.6052 35.56 0)
+			(at 164.7952 35.56 0)
 			(effects
 				(font
@@
 		)
 		(property "Datasheet" "~"
-			(at 167.64 31.75 0)
+			(at 163.83 31.75 0)
 			(effects
 				(font
@@
 		)
 		(property "Description" "Unpolarized capacitor"
-			(at 167.64 31.75 0)
+			(at 163.83 31.75 0)
 			(effects
 				(font
@@
 	)
 	(symbol
+		(lib_id "Device:C")
+		(at 170.18 31.75 0)
+		(unit 1)
+		(exclude_from_sim no)
+		(in_bom yes)
+		(on_board yes)
+		(dnp no)
+		(property "Reference" "C10"
+			(at 165.862 29.21 0)
+			(effects
+				(font
+					(size 1.27 1.27)
+				)
+				(justify left)
+			)
+		)
+		(property "Value" "100n"
+			(at 165.1 34.036 0)
+			(effects
+				(font
+					(size 1.27 1.27)
+				)
+				(justify left)
+			)
+		)
+		(property "Footprint" "Capacitor_SMD:C_0805_2012Metric"
+			(at 171.1452 35.56 0)
+			(effects
+				(font
+					(size 1.27 1.27)
+				)
+				(hide yes)
+			)
+		)
+		(property "Datasheet" "~"
+			(at 170.18 31.75 0)
+			(effects
+				(font
+					(size 1.27 1.27)
+				)
+				(hide yes)
+			)
+		)
+		(property "Description" "Unpolarized capacitor"
+			(at 170.18 31.75 0)
+			(effects
+				(font
+					(size 1.27 1.27)
+				)
+				(hide yes)
+			)
+		)
+		(pin "2"
+		)
+		(pin "1"
+		)
+		(instances
+			(project "FCU_v1"
+				(path "/ace60bf5-8c2a-49e8-98f3-824f03a0dfeb/59ff9d4e-fbb6-4b08-8a4a-edebb7815a6e"
+					(reference "C10")
+					(unit 1)
+				)
+			)
+		)
+	)
+	(symbol
 		(lib_id "Power_Protection:USBLC6-2SC6")
 		(at 69.85 147.32 0)
@@
 	(symbol
 		(lib_id "power:GND")
-		(at 167.64 36.83 0)
+		(at 163.83 38.1 0)
 		(unit 1)
 		(exclude_from_sim no)
@@
 		(fields_autoplaced yes)
 		(property "Reference" "#PWR022"
-			(at 167.64 43.18 0)
+			(at 163.83 44.45 0)
 			(effects
 				(font
@@
 		)
 		(property "Value" "GND"
-			(at 167.64 41.91 0)
+			(at 163.83 43.18 0)
 			(effects
 				(font
@@
 		)
 		(property "Footprint" ""
-			(at 167.64 36.83 0)
+			(at 163.83 38.1 0)
 			(effects
 				(font
@@
 		)
 		(property "Datasheet" ""
-			(at 167.64 36.83 0)
+			(at 163.83 38.1 0)
 			(effects
 				(font
@@
 		)
 		(property "Description" "Power symbol creates a global label with name \"GND\" , ground"
-			(at 167.64 36.83 0)
+			(at 163.83 38.1 0)
 			(effects
 				(font
