File: PCB/FCU_v1/FCU_v1.kicad_pcb (KiCad board)
At the start: 4 copper layers, 57.6 x 60.8 mm, 109 parts, among them J1 Conn_01x04_Pin, J10 Conn_01x04_Pin, J11 USB_C_Receptacle_USB2.0_16P, J3 Conn_01x05_Pin, J4 Conn_Coaxial_Small, J5 Conn_01x04_Pin, J6 Conn_01x04_Pin, J7 Conn_01x04_Pin, J8 Conn_01x04_Pin, J9 Conn_01x04_Pin, U1 TPS62132, U10 SN65HVD232, U11 STM32G473RETx, U3 TLV75533PDYDR, U4 BMI088, U5 LIS2MDL, U6 LPS22HH, U7 W25Q64JV, U8 USBLC6-2SC6, U9 MAX-M10M-20B, Y2 16MHz

Commit message: Layout update
Parts:
- removed C10, C32: 100n, Capacitor_SMD:C_0805_2012Metric
- removed C35: 4u7-10u, Capacitor_SMD:C_0805_2012Metric
- removed D4: LED, LED_SMD:LED_0805_2012Metric
- removed J4: Conn_Coaxial_Small, Connector_Coaxial:SMA_Amphenol_901-143_Horizontal
- removed R13, R14, R23: 33R, Resistor_SMD:R_0603_1608Metric
- removed R15: 4.7k, Resistor_SMD:R_0603_1608Metric
- removed R16: 10k/DNP, Resistor_SMD:R_0603_1608Metric
- removed U9: MAX-M10M-20B, RF_GPS:ublox_MAX
Routing:
- net GNSS_TX: track 32.6 -> 0.00 mm
- net GNSS_RX: track 26.5 -> 0.00 mm
- net Net-(U9-TIMEPULSE): track 9.17 -> 0.00 mm
- net 3V3_FCU: track 22.9 -> 13.8 mm
- net GND: track 24.6 -> 20.7 mm
- net Net-(U9-TXD): track 3.62 -> 0.00 mm
- net Net-(D4-A): track 1.52 -> 0.00 mm
Other:
- outline, holes or cut-outs redrawn

Commit message: Schematic update
Parts:
- removed C23: 220n, Capacitor_SMD:C_0805_2012Metric
- removed C24, C25, C27, C29: 100n, Capacitor_SMD:C_0805_2012Metric
- removed C26, C28: 10u, Capacitor_SMD:C_0805_2012Metric
- removed D2: LED, LED_SMD:LED_0805_2012Metric
- removed D7: SMAJ5.0CA, Diode_SMD:D_SMA
- removed L2: 2.2uH, Inductor_SMD:L_Coilcraft_XxL4020
- removed R31, R34: 33R, Resistor_SMD:R_0603_1608Metric
- removed R6: 4.7k, Resistor_SMD:R_0603_1608Metric
- removed R7, R8: DNP, Resistor_SMD:R_0201_0603Metric
- removed U5: LIS2MDL, Package_LGA:LGA-12_2x2mm_P0.5mm
- removed U6: LPS22HH, Package_LGA:ST_HLGA-10_2x2mm_P0.5mm_LayoutBorder3x2y
- removed U7: W25Q64JV, Package_SO:SOIC-8_5.3x5.3mm_P1.27mm
- added C36: 2u2, Capacitor_SMD:C_0805_2012Metric, F.Cu at (184.0, 111.4)
- added C38: 1u, Capacitor_SMD:C_0805_2012Metric, F.Cu at (184.0, 114.4)
- added C39: 100n, Capacitor_SMD:C_0805_2012Metric, F.Cu at (184.0, 117.5)
- added C40: 100n, Capacitor_SMD:C_0805_2012Metric, F.Cu at (184.0, 120.5)
- added C42: 2u2, Capacitor_SMD:C_0805_2012Metric, F.Cu at (184.0, 123.5)
- added D9: ESD2CAN24DBZRQ1, Package_TO_SOT_SMD:SOT-23-3, F.Cu at (199.6, 105.2)
- added IC1: BMM350, SamacSys_Parts:BGA9C40P3X3_128X128X54, F.Cu at (194.9, 112.1)
- added IC2: TPS7A2018PDBVR, SamacSys_Parts:SOT95P280X145-5N, F.Cu at (188.9, 124.8)
- added IC3: ESP32-C3-MINI-1-N4X, SamacSys_Parts:ESP32C3MINI1N4X, F.Cu at (216.3, 111.0)
- added L1: 744042001, SamacSys_Parts:WE-TPC_4818_482892, F.Cu at (225.6, 89.2)
- added R37: 100k, Resistor_SMD:R_0603_1608Metric, F.Cu at (210.2, 91.7)
- added R38: DNP, Resistor_SMD:R_0201_0603Metric, F.Cu at (191.5, 110.8)
- added R39: DNP, Resistor_SMD:R_0201_0603Metric, F.Cu at (191.5, 112.6)
- added R41: DNP, Resistor_SMD:R_0201_0603Metric, F.Cu at (191.5, 114.3)
- added R42: DNP, Resistor_SMD:R_0201_0603Metric, F.Cu at (191.5, 116.1)
- added U2: BMP581, SamacSys_Parts:BMP581, F.Cu at (194.1, 125.0)
- C1: value 3.3nF -> 22u/10V
- C15, C17, C20, C22, C31, D3, FB2, R10, R11, R12, R27, R28, R29, R3, R30, R9: moved to F.Cu
- C18: value 2u2/4u7 -> 100n; moved to F.Cu
- C19: value 2u2 -> 100n; moved to F.Cu
- C2: value 22uF -> 100n/10V
- C3: value 0.1uF -> 2u2/6.3V
- C30: value 10u -> 2u2
- C4: value 10uF -> 10u/10V
- R1: value 100k -> 2k
- R2: value 4.7k -> 450k
- U1: value TPS62132 -> TPS62A02APDDCR; footprint Package_DFN_QFN:VQFN-16-1EP_3x3mm_P0.5mm_EP1.68x1.68mm_ThermalVias -> Package_TO_SOT_SMD:SOT-23-6
- U3: value TLV75533PDYDR -> W25Q128JVSIM; footprint Package_TO_SOT_SMD:SOT-23-5_HandSoldering -> Package_SO:SOIC-8_5.3x5.3mm_P1.27mm; moved to F.Cu
- moved D3 111.9 mm to (219.0, 96.6)
- moved FB2 104.6 mm to (224.1, 97.8), turned to 0 degrees
- moved D6 101.0 mm to (224.7, 94.7), turned to 0 degrees
- moved J11 99.6 mm to (222.5, 80.7)
- moved C17 97.4 mm to (214.4, 86.0)
- moved C20 96.4 mm to (214.4, 89.0)
- moved R11 93.8 mm to (205.0, 86.7), turned to 0 degrees
- moved R12 92.9 mm to (205.0, 88.5), turned to 0 degrees
- moved U3 91.9 mm to (200.5, 79.0), turned to 0 degrees
- moved U8 90.9 mm to (219.2, 92.4), turned to 0 degrees
- moved R36 90.9 mm to (210.2, 89.2), turned to 0 degrees
- moved U4 89.4 mm to (193.4, 119.7), turned to 0 degrees
- moved J3 89.0 mm to (193.0, 77.7)
- moved R9 87.6 mm to (205.0, 83.2), turned to 0 degrees
- moved R10 87.5 mm to (205.0, 85.0)
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Connections:
- net /PERIPHERALS/D+ renamed /D+
- net /PERIPHERALS/D- renamed /D-
- net /PERIPHERALS/USB_VBUS renamed /USB_VBUS
- C1 pad 1: Net-(U1-SS/TR) -> +3.3V
- C17 pad 1: VBUS -> +VBUS
- C18 pad 1: VBUS -> Net-(IC1-VDD)
- C19 pad 1: VBUS_3V3 -> +3.3V
- C2 pad 1: 3V3 -> +5V_FCU
- C20 pad 1: VBUS -> +VBUS
- C21 pad 1: 3V3_FCU -> +3.3V
- C22 pad 1: 3V3_FCU -> +3.3V
- C3 pad 1: 5V_PDU -> Net-(IC1-CRST)
- C30 pad 1: 3V3_FCU -> +3.3V
- C31 pad 1: 3V3_FCU -> +3.3V
- C33 pad 1: 3V3 -> +3.3V
- C34 pad 1: 3V3 -> +3.3V
- C4 pad 1: 5V_PDU -> +5V_FCU
- D3 pad 1: VBUS_3V3 -> +VBUS
- D3 pad 2: 3V3 -> +5V
- D3 pad 3: 3V3_FCU -> +5V_FCU
- FB2 pad 2: VBUS -> +VBUS
- J1 pad 1: 5V_PDU -> +5V
- J10 pad 1: 3V3 -> +5V
- J3 pad 1: 3V3_FCU -> +3.3V
- J5 pad 1: 3V3 -> +5V
- J6 pad 1: 3V3 -> +5V
- J7 pad 1: 3V3 -> +5V
- J8 pad 1: 3V3 -> +5V
- J9 pad 1: 3V3 -> +5V
- R1 pad 1: 3V3 -> +3.3V
- R1 pad 2: Net-(U1-PG) -> Net-(D1-A)
- R10 pad 2: Net-(U7-~{WP}/IO_{2}) -> Net-(U3-~{WP}/IO_{2})
- R11 pad 2: Net-(U7-~{HOLD}/~{RESET}/IO_{3}) -> Net-(U3-~{HOLD}/~{RESET}/IO_{3})
- R12 pad 1: Net-(U7-~{HOLD}/~{RESET}/IO_{3}) -> Net-(U3-~{HOLD}/~{RESET}/IO_{3})
- R12 pad 2: 3V3_FCU -> +3.3V
- R2 pad 1: 3V3 -> +3.3V
- R2 pad 2: Net-(D1-A) -> Net-(U1-FB)
- R22 pad 2: Net-(U7-DO/IO_{1}) -> Net-(U3-DO/IO_{1})
- R4 pad 2: VBUS -> +VBUS
- R9 pad 1: Net-(U7-~{WP}/IO_{2}) -> Net-(U3-~{WP}/IO_{2})
- R9 pad 2: 3V3_FCU -> +3.3V
- U1 pad 1: /BUCK_SW -> +5V_FCU
- U1 pad 2: /BUCK_SW -> GND
- U1 pad 3: /BUCK_SW -> Net-(U1-SW)
- U1 pad 4: Net-(U1-PG) -> +5V_FCU
- U1 pad 6: GND -> Net-(U1-FB)
- U10 pad 3: 3V3 -> +3.3V
- U11 pad 58: /MCU/GNSS_Rst -> unconnected-(U11-PB5-Pad58)
- U11 pad 59: /MCU/GNSS_Tx -> unconnected-(U11-PB6-Pad59)
- U3 pad 1: VBUS -> CS_MEMO
- U3 pad 2: GND -> Net-(U3-DO/IO_{1})
- U3 pad 3: VBUS -> Net-(U3-~{WP}/IO_{2})
- U3 pad 4: unconnected-(U3-NC-Pad4) -> GND
- U3 pad 5: VBUS_3V3 -> SPI_MOSI
- U4 pad 11: 3V3_FCU -> +3.3V
- U4 pad 3: 3V3_FCU -> +3.3V
Routing:
- net 3V3: track 142.4 -> 0.00 mm, vias 8 -> 0
- net BAT_CURR: track 32.1 -> 0.00 mm
- net BAT_VOL: track 28.4 -> 0.00 mm
- net SPI_SCK: track 22.7 -> 0.00 mm
- net GND: track 20.7 -> 0.00 mm, vias 2 -> 0
- net INT1_ACCEL: track 19.1 -> 0.00 mm, vias 1 -> 0
- net SPI_MISO: track 15.5 -> 0.00 mm
- net 3V3_FCU: track 13.8 -> 0.00 mm, vias 2 -> 0
- net SPI_MOSI: track 12.1 -> 0.00 mm
- net CSB_GYRO: track 11.7 -> 0.00 mm, vias 1 -> 0
- net Net-(U4-SDO1): track 11.3 -> 0.00 mm
- net OSC_IN: track 11.1 -> 0.00 mm
- net INT2_ACCEL: track 11.0 -> 0.00 mm, vias 1 -> 0
- net VBUS_3V3: track 10.1 -> 0.00 mm
- net OSC_OUT: track 7.34 -> 0.00 mm
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- removed copper zone on F.Cu, net /BUCK_SW
- removed copper zone on F.Cu, net 3V3
- removed copper zone on F.Cu, net 5V_PDU
- removed copper zone on F.Cu, net GND

Commit message: Repaired library
Parts:
- removed IC1: BMM350, SamacSys_Parts:BGA9C40P3X3_128X128X54
- removed U2: BMP581, SamacSys_Parts:BMP581
- added C37: 10u, Capacitor_SMD:C_0805_2012Metric, F.Cu at (221.4, 125.0)
- added C43: 100n, Capacitor_SMD:C_0805_2012Metric, F.Cu at (221.4, 128.0)
- added C44: 1u, Capacitor_SMD:C_0805_2012Metric, F.Cu at (221.4, 131.0)
- added C45: 100n, Capacitor_SMD:C_0805_2012Metric, F.Cu at (221.4, 134.0)
- added D2: LED, LED_SMD:LED_0805_2012Metric, F.Cu at (225.9, 132.5)
- added IC4: ESP32-C3-MINI-1-N4X, SamacSys_Parts:ESP32C3MINI1N4X, F.Cu at (211.1, 116.7)
- added R44: 10k, Resistor_SMD:R_0603_1608Metric, F.Cu at (225.7, 124.7)
- added R45: 10k, Resistor_SMD:R_0603_1608Metric, F.Cu at (225.7, 127.2)
- added R46: 2k, Resistor_SMD:R_0603_1608Metric, F.Cu at (225.7, 129.7)
- added SW3: SW_MEC_5G, Button_Switch_SMD:SW_MEC_5GSH9, F.Cu at (225.0, 115.1)
- added U7: BMP581, SamacSys_Parts:BMP581, F.Cu at (235.4, 114.0)
- IC2: value TPS7A2018PDBVR -> BMM350; footprint SamacSys_Parts:SOT95P280X145-5N -> SamacSys_Parts:BGA9C40P3X3_128X128X54
- IC3: value ESP32-C3-MINI-1-N4X -> TPS7A2018PDBVR; footprint SamacSys_Parts:ESP32C3MINI1N4X -> SamacSys_Parts:SOT95P280X145-5N
- moved IC2 52.5 mm to (240.1, 113.6)
- moved L1 32.1 mm to (235.6, 119.7)
- moved IC3 19.2 mm to (235.5, 109.1)
Connections:
- net STM_VDDA renamed +3.3VA
- C1 pad 1: +3.3V -> STM_VDD
- C11 pad 1: 3V3_FCU -> STM_VDD
- C14 pad 1: 3V3_FCU -> STM_VDD
- C18 pad 1: Net-(IC1-VDD) -> Net-(IC2-VDD)
- C19 pad 1: +3.3V -> STM_VDD
- C21 pad 1: +3.3V -> STM_VDD
- C22 pad 1: +3.3V -> STM_VDD
- C3 pad 1: Net-(IC1-CRST) -> Net-(IC2-CRST)
- C30 pad 1: +3.3V -> STM_VDD
- C31 pad 1: +3.3V -> STM_VDD
- C33 pad 1: +3.3V -> STM_VDD
- C34 pad 1: +3.3V -> STM_VDD
- C36 pad 1: Net-(IC1-VDD) -> Net-(IC2-VDD)
- C38 pad 1: +3.3V -> STM_VDD
- C39 pad 1: +3.3V -> STM_VDD
- C40 pad 1: +3.3V -> STM_VDD
- C42 pad 1: +3.3V -> STM_VDD
- C5 pad 1: 3V3_FCU -> STM_VDD
- C6 pad 1: 3V3_FCU -> STM_VDD
- C7 pad 1: 3V3_FCU -> STM_VDD
- C8 pad 1: 3V3_FCU -> STM_VDD
- C9 pad 1: 3V3_FCU -> STM_VDD
- FB1 pad 2: 3V3_FCU -> STM_VDD
- IC3 pad 1: GND -> STM_VDD
- IC3 pad 3: unconnected-(IC3-3V3-Pad3) -> STM_VDD
- IC3 pad 5: unconnected-(IC3-IO2-Pad5) -> Net-(IC2-VDD)
- J3 pad 1: +3.3V -> STM_VDD
- L1 pad 2: +3.3V -> STM_VDD
- R1 pad 1: +3.3V -> STM_VDD
- R12 pad 2: +3.3V -> STM_VDD
- R17 pad 1: I2C_SCL -> STM_VDD
- R17 pad 2: 3V3_FCU -> I2C_SCL
- R18 pad 1: I2C_SDA -> STM_VDD
- R18 pad 2: 3V3_FCU -> I2C_SDA
- R2 pad 1: +3.3V -> STM_VDD
- R38 pad 1: Net-(IC1-ADSEL) -> Net-(IC2-ADSEL)
- R39 pad 1: +3.3V -> STM_VDD
- R39 pad 2: Net-(IC1-ADSEL) -> Net-(IC2-ADSEL)
- R41 pad 1: +3.3V -> STM_VDD
- R9 pad 2: +3.3V -> STM_VDD
- U10 pad 3: +3.3V -> STM_VDD
- U11 pad 1: 3V3_FCU -> STM_VDD
- U11 pad 16: 3V3_FCU -> STM_VDD
- U11 pad 32: 3V3_FCU -> STM_VDD
- U11 pad 48: 3V3_FCU -> STM_VDD
- U11 pad 64: 3V3_FCU -> STM_VDD
- U3 pad 8: +3.3V -> STM_VDD
- U4 pad 11: +3.3V -> STM_VDD
- U4 pad 3: +3.3V -> STM_VDD
