File: PCB/FCU_v1/MCU.kicad_sch (KiCad schematic)
At the start: 51 parts, among them J12 Conn_01x02_Pin, J13 Conn_01x02_Pin, J3 Conn_01x02_Pin, U10 SN65HVD232, U2 STM32F412RETx, U3 W25Q128JVSIM, Y2 16MHz

Commit message: Layout update
Parts:
- added IC2: TCAN3414DR, SOIC127P600X175-8N, symbol SamacSys_Parts:TCAN3414DR
- C16, C41: value 10p -> 6p8; footprint Capacitor_SMD:C_0805_2012Metric -> Capacitor_SMD:C_0603_1608Metric
- C34: footprint Capacitor_SMD:C_0805_2012Metric -> Capacitor_SMD:C_0603_1608Metric
- FB1: value 120R at 100 MHz -> FCM1608KF-601T03; footprint Inductor_SMD:L_0805_2012Metric -> Inductor_SMD:L_0603_1608Metric
- R10, R11, R12, R39, R9: footprint Resistor_SMD:R_0201_0603Metric -> Resistor_SMD:R_0402_1005Metric
- Y2: value 16MHz -> 24MHz
Other:
- note added: "ABM8W-24.0000MHZ-6-D1X-T3"
- note added: "FCM1608KF-601T03 600 Ω @ 100 MHz, low DC resistance From ST datasheet and BOM"
- note added: "Values from STM's G4 Nucleo Board Schematic"
- note removed: "120R at 100 MHz"
